Commit message: To jetson

File: ros2_ws/src/robot_description/urdf/Robot.xacro (robot description, xacro)
@@ -4,13 +4,19 @@
 <xacro:include filename="$(find robot_description)/urdf/Robot.trans" />
 <xacro:include filename="$(find robot_description)/urdf/Robot.gazebo" />
-<!-- REP-103/105 driving frame: X forward, Z up. The estimator publishes
-     odom->base_link, so this frame must stay axis-aligned. The Fusion model is
-     mounted under it via a fixed joint that applies the -90 deg roll about X
-     (clockwise looking down +X) needed to stand the mesh upright, WITHOUT
-     tilting the odometry frame. Flip the sign of the roll if it rotates the
-     wrong way. Root link is empty (no inertia) so KDL emits no warning. -->
+<!-- REP-103/105 driving frame: X forward, +Y left, Z up. The estimator publishes
+     odom->base_link, so this frame must stay axis-aligned. The chassis mesh is
+     mounted under it via a fixed joint that applies the +90 deg roll about X
+     needed to stand the mesh upright, WITHOUT tilting the odometry frame.
+     Flip the sign of the roll if it rotates the wrong way. Root link is empty
+     (no inertia) so KDL emits no warning.
+     The xyz translation places base_link at the DRIVE-WHEEL AXLE MIDPOINT (the
+     differential-drive kinematic center the estimator integrates), not the CAD
+     origin. It is -1 * (axle midpoint expressed in base_link); with it the two
+     wheels sit symmetric at Y = +/-0.146 m, X~=0, Z~=0. Recompute if the wheel
+     joint origins change: take the mean of the two Revolution joint origins
+     (chassis frame), map (x,y,z)->(x,-z,y), and negate. -->
 <link name="base_link"/>
 <joint name="base_mount" type="fixed">
-  <origin xyz="0 0 0" rpy="1.5708 0 0"/>
+  <origin xyz="0.018885 -0.125267 -0.034371" rpy="1.5708 0 0"/>
   <parent link="base_link"/>
   <child link="chassis"/>
@@ -84,3 +90,15 @@
   <axis xyz="0.0 -0.0 1.0"/>
 </joint>
+<!-- IMU (OAK-D) mount, relative to base_link (the axle center). Offsets are from
+     CAD, measured from the wheel-axle midpoint: 0.42 m forward (X), 0.135 m up (Z),
+     centered on width (Y = 0). Translation is placement only — it does NOT affect
+     orientation fusion (we fuse roll/pitch/yaw-rate, not linear accel). The camera
+     is mounted level (no tilt), so rpy = 0: its REP-103-remapped axes align with
+     base_link and a level robot reports ~0 roll/pitch (in complementary mode). -->
+<link name="imu_link"/>
+<joint name="imu_mount" type="fixed">
+  <origin xyz="0.42 0 0.135" rpy="0 0 0"/>
+  <parent link="base_link"/>
+  <child link="imu_link"/>
+</joint>
 </robot>

Commit message: EKF

File: ros2_ws/src/robot_description/urdf/Robot.xacro (robot description, xacro)
@@ -102,3 +102,15 @@
   <child link="imu_link"/>
 </joint>
+<!-- RPLidar A1M8 — centered on robot (x=0, y=0), mounted at the top.
+     Z=0.20 m is measured from the wheel-axle midpoint (base_link origin).
+     ADJUST Z if the actual mount height differs — measure from axle to lidar
+     scan plane in metres. The lidar sits flat (no roll/pitch), facing forward
+     (no yaw offset). Frame name "laser" matches sllidar_ros2's default frame_id
+     so no remapping is needed. -->
+<link name="laser"/>
+<joint name="lidar_mount" type="fixed">
+  <origin xyz="0.0 0.0 0.20" rpy="0 0 0"/>
+  <parent link="base_link"/>
+  <child link="laser"/>
+</joint>
 </robot>

Commit message: moving stuff

File: ros2_ws/src/robot_description/urdf/Robot.xacro (robot description, xacro)
@@ -47,5 +47,5 @@
     <origin xyz="0.018502 -0.032756 0.27162" rpy="0 0 0"/>
     <geometry>
-      <mesh filename="package://robot_description/meshes/Moteur_+_Roue_v1_Symetrie_miroir__1.stl" scale="0.001 0.001 0.001"/>
+      <mesh filename="package://robot_description/meshes/Moteur_+_Roue_v1_Symétrie_miroir__1.stl" scale="0.001 0.001 0.001"/>
     </geometry>
     <material name="silver"/>
@@ -54,5 +54,5 @@
     <origin xyz="0.018502 -0.032756 0.27162" rpy="0 0 0"/>
     <geometry>
-      <mesh filename="package://robot_description/meshes/Moteur_+_Roue_v1_Symetrie_miroir__1.stl" scale="0.001 0.001 0.001"/>
+      <mesh filename="package://robot_description/meshes/Moteur_+_Roue_v1_Symétrie_miroir__1.stl" scale="0.001 0.001 0.001"/>
     </geometry>
   </collision>
@@ -110,5 +110,5 @@
 <link name="laser"/>
 <joint name="lidar_mount" type="fixed">
-  <origin xyz="0.0 0.0 0.20" rpy="0 0 0"/>
+  <origin xyz="0.280 -0.040 0.211" rpy="0 0 0"/>
   <parent link="base_link"/>
   <child link="laser"/>

Commit message: refactor: switches some custom nodes for field tested packages

File: ros2_ws/src/robot_description/urdf/Robot.xacro (robot description, xacro)
@@ -78,16 +78,40 @@
   </collision>
 </link>
-<joint name="Revolution 3" type="continuous">
+<joint name="left_wheel_joint" type="continuous">
   <origin xyz="-0.018502 0.032756 -0.27162" rpy="0 0 0"/>
   <parent link="chassis"/>
   <child link="Moteur_+_Roue_v1_Symetrie_miroir__1"/>
-  <axis xyz="-0.0 0.0 1.0"/>
+  <axis xyz="0.0 0.0 1.0"/>
 </joint>
-<joint name="Revolution 4" type="continuous">
+<joint name="right_wheel_joint" type="continuous">
   <origin xyz="-0.019268 0.035986 0.021086" rpy="0 0 0"/>
   <parent link="chassis"/>
   <child link="Moteur_+_Roue_v3_1"/>
-  <axis xyz="0.0 -0.0 1.0"/>
+  <axis xyz="0.0 0.0 1.0"/>
 </joint>
+<!-- ros2_control block: hardware interface plugin + joint interfaces.
+     Parameters mirror state_estimator_node.py and cmd_vel_bridge_node.py. -->
+<ros2_control name="eyerobot_hardware" type="system">
+  <hardware>
+    <plugin>eyerobot_hardware/EyeRobotHardware</plugin>
+    <param name="counts_per_output_rev">5756.0</param>
+    <param name="right_feedback_sign">1.0</param>
+    <param name="left_feedback_sign">-1.0</param>
+    <param name="right_fb_topic">motor_rwheel_fb</param>
+    <param name="left_fb_topic">motor_lwheel_fb</param>
+    <param name="right_cmd_topic">motor_rwheel_cmd</param>
+    <param name="left_cmd_topic">motor_lwheel_cmd</param>
+  </hardware>
+  <joint name="right_wheel_joint">
+    <command_interface name="velocity"/>
+    <state_interface name="position"/>
+    <state_interface name="velocity"/>
+  </joint>
+  <joint name="left_wheel_joint">
+    <command_interface name="velocity"/>
+    <state_interface name="position"/>
+    <state_interface name="velocity"/>
+  </joint>
+</ros2_control>
 <!-- IMU (OAK-D) mount, relative to base_link (the axle center). Offsets are from
      CAD, measured from the wheel-axle midpoint: 0.42 m forward (X), 0.135 m up (Z),

Commit message: test

File: ros2_ws/src/robot_description/urdf/Robot.xacro (robot description, xacro)
@@ -129,4 +129,14 @@
   <child link="imu_link"/>
 </joint>
+<!-- depthai_ros_driver stamps IMU messages with frame_id oak_imu_frame, but the
+     driver's own URDF (oak_state_publisher) does not include that frame unless
+     imu_from_descr is enabled — so robot_localization could not transform the
+     IMU data. Provide it here: same pose as imu_link (the OAK-D IS the IMU). -->
+<link name="oak_imu_frame"/>
+<joint name="oak_imu_mount" type="fixed">
+  <origin xyz="0 0 0" rpy="0 0 0"/>
+  <parent link="imu_link"/>
+  <child link="oak_imu_frame"/>
+</joint>
 <!-- RPLidar A1M8 — centered on robot (x=0, y=0), mounted at the top.
      Z=0.20 m is measured from the wheel-axle midpoint (base_link origin).

Commit message: t

File: ros2_ws/src/robot_description/urdf/Robot.xacro (robot description, xacro)
@@ -133,7 +133,12 @@
      imu_from_descr is enabled — so robot_localization could not transform the
      IMU data. Provide it here: same pose as imu_link (the OAK-D IS the IMU). -->
+<!-- rpy = (pi,0,0): the OAK-D's IMU frame is rolled 180 deg vs REP-103 — its
+     +z gyro reads NEGATIVE on a counter-clockwise (left) robot turn. Verified
+     on hardware: with rpy 0 the EKF turned right when the robot turned left.
+     Equivalent to the old imu_remap_node gyro_signs [1,-1,-1]; encoding it in
+     the frame lets robot_localization rotate the rates instead. -->
 <link name="oak_imu_frame"/>
 <joint name="oak_imu_mount" type="fixed">
-  <origin xyz="0 0 0" rpy="0 0 0"/>
+  <origin xyz="0 0 0" rpy="3.141592653589793 0 0"/>
   <parent link="imu_link"/>
   <child link="oak_imu_frame"/>

Commit message: test new

File: ros2_ws/src/robot_description/urdf/Robot.xacro (robot description, xacro)
@@ -129,19 +129,9 @@
   <child link="imu_link"/>
 </joint>
-<!-- depthai_ros_driver stamps IMU messages with frame_id oak_imu_frame, but the
-     driver's own URDF (oak_state_publisher) does not include that frame unless
-     imu_from_descr is enabled — so robot_localization could not transform the
-     IMU data. Provide it here: same pose as imu_link (the OAK-D IS the IMU). -->
-<!-- rpy = (pi,0,0): the OAK-D's IMU frame is rolled 180 deg vs REP-103 — its
-     +z gyro reads NEGATIVE on a counter-clockwise (left) robot turn. Verified
-     on hardware: with rpy 0 the EKF turned right when the robot turned left.
-     Equivalent to the old imu_remap_node gyro_signs [1,-1,-1]; encoding it in
-     the frame lets robot_localization rotate the rates instead. -->
-<link name="oak_imu_frame"/>
-<joint name="oak_imu_mount" type="fixed">
-  <origin xyz="0 0 0" rpy="3.141592653589793 0 0"/>
-  <parent link="imu_link"/>
-  <child link="oak_imu_frame"/>
-</joint>
+<!-- IMU data is published in imu_link directly: imu_remap_node corrects the
+     BMI270's 180°-about-X mounting in the DATA (gyro/accel signs) and stamps
+     frame_id imu_link. A TF-level fix (oak_imu_frame rolled by pi) was tried
+     and abandoned — robot_localization did not flip the integrated yaw rate
+     despite the transform being live (hardware-verified 2026-06-10). -->
 <!-- RPLidar A1M8 — centered on robot (x=0, y=0), mounted at the top.
      Z=0.20 m is measured from the wheel-axle midpoint (base_link origin).

Commit message: cleaned and URDF try on foxglove

File: ros2_ws/src/robot_description/urdf/Robot.xacro (robot description, xacro)
@@ -38,5 +38,5 @@
   </collision>
 </link>
-<link name="Moteur_+_Roue_v1_Symetrie_miroir__1">
+<link name="left_wheel_link">
   <inertial>
     <origin xyz="5.182027081260254e-07 3.7287997872448297e-06 -0.021890971794159053" rpy="0 0 0"/>
@@ -47,5 +47,5 @@
     <origin xyz="0.018502 -0.032756 0.27162" rpy="0 0 0"/>
     <geometry>
-      <mesh filename="package://robot_description/meshes/Moteur_+_Roue_v1_Symétrie_miroir__1.stl" scale="0.001 0.001 0.001"/>
+      <mesh filename="package://robot_description/meshes/wheel_mirrored.stl" scale="0.001 0.001 0.001"/>
     </geometry>
     <material name="silver"/>
@@ -54,9 +54,9 @@
     <origin xyz="0.018502 -0.032756 0.27162" rpy="0 0 0"/>
     <geometry>
-      <mesh filename="package://robot_description/meshes/Moteur_+_Roue_v1_Symétrie_miroir__1.stl" scale="0.001 0.001 0.001"/>
+      <mesh filename="package://robot_description/meshes/wheel_mirrored.stl" scale="0.001 0.001 0.001"/>
     </geometry>
   </collision>
 </link>
-<link name="Moteur_+_Roue_v3_1">
+<link name="right_wheel_link">
   <inertial>
     <origin xyz="-9.7522353499635e-07 3.924730006502064e-06 0.02189068703142081" rpy="0 0 0"/>
@@ -67,5 +67,5 @@
     <origin xyz="0.019268 -0.035986 -0.021086" rpy="0 0 0"/>
     <geometry>
-      <mesh filename="package://robot_description/meshes/Moteur_+_Roue_v3_1.stl" scale="0.001 0.001 0.001"/>
+      <mesh filename="package://robot_description/meshes/wheel.stl" scale="0.001 0.001 0.001"/>
     </geometry>
     <material name="silver"/>
@@ -74,5 +74,5 @@
     <origin xyz="0.019268 -0.035986 -0.021086" rpy="0 0 0"/>
     <geometry>
-      <mesh filename="package://robot_description/meshes/Moteur_+_Roue_v3_1.stl" scale="0.001 0.001 0.001"/>
+      <mesh filename="package://robot_description/meshes/wheel.stl" scale="0.001 0.001 0.001"/>
     </geometry>
   </collision>
@@ -81,5 +81,5 @@
   <origin xyz="-0.018502 0.032756 -0.27162" rpy="0 0 0"/>
   <parent link="chassis"/>
-  <child link="Moteur_+_Roue_v1_Symetrie_miroir__1"/>
+  <child link="left_wheel_link"/>
   <axis xyz="0.0 0.0 1.0"/>
 </joint>
@@ -87,5 +87,5 @@
   <origin xyz="-0.019268 0.035986 0.021086" rpy="0 0 0"/>
   <parent link="chassis"/>
-  <child link="Moteur_+_Roue_v3_1"/>
+  <child link="right_wheel_link"/>
   <axis xyz="0.0 0.0 1.0"/>
 </joint>
@@ -119,8 +119,8 @@
 <!-- IMU (OAK-D) mount, relative to base_link (the axle center). Offsets are from
      CAD, measured from the wheel-axle midpoint: 0.42 m forward (X), 0.135 m up (Z),
-     centered on width (Y = 0). Translation is placement only — it does NOT affect
-     orientation fusion (we fuse roll/pitch/yaw-rate, not linear accel). The camera
-     is mounted level (no tilt), so rpy = 0: its REP-103-remapped axes align with
-     base_link and a level robot reports ~0 roll/pitch (in complementary mode). -->
+     centered on width (Y = 0). NOTE: the physical camera is TILTED ~58° from
+     vertical (looking at the floor) — imu_remap_node measures that tilt from
+     gravity at startup and rotates the IMU data into this level, body-aligned
+     frame, so imu_link stays rpy = 0 here and the data matches it. -->
 <link name="imu_link"/>
 <joint name="imu_mount" type="fixed">
